Commit message: Make all 2F-85 joints revolute

File: robotiq_description/urdf/robotiq_2f_85_macro.urdf.xacro (robot description, xacro)
@@ -257,5 +257,5 @@
             <origin xyz="-0.03152616 0.0 -0.00376347" rpy="0 0 0" />
         </joint>
-        <joint name="${prefix}robotiq_85_left_inner_knuckle_joint" type="continuous">
+        <joint name="${prefix}robotiq_85_left_inner_knuckle_joint" type="revolute">
             <parent link="${prefix}robotiq_85_base_link" />
             <child link="${prefix}robotiq_85_left_inner_knuckle_link" />
@@ -263,6 +263,7 @@
             <origin xyz="0.0127 0.0 0.06142" rpy="0 0 0" />
             <mimic joint="${prefix}robotiq_85_left_knuckle_joint" />
-        </joint>
-        <joint name="${prefix}robotiq_85_right_inner_knuckle_joint" type="continuous">
+            <limit lower="0.0" upper="0.8" velocity="0.5" effort="50" />
+        </joint>
+        <joint name="${prefix}robotiq_85_right_inner_knuckle_joint" type="revolute">
             <parent link="${prefix}robotiq_85_base_link" />
             <child link="${prefix}robotiq_85_right_inner_knuckle_link" />
@@ -270,6 +271,7 @@
             <origin xyz="-0.0127 0.0 0.06142" rpy="0 0 0" />
             <mimic joint="${prefix}robotiq_85_left_knuckle_joint" multiplier="-1" />
-        </joint>
-        <joint name="${prefix}robotiq_85_left_finger_tip_joint" type="continuous">
+            <limit lower="-0.8" upper="0.0" velocity="0.5" effort="50" />
+        </joint>
+        <joint name="${prefix}robotiq_85_left_finger_tip_joint" type="revolute">
             <parent link="${prefix}robotiq_85_left_finger_link" />
             <child link="${prefix}robotiq_85_left_finger_tip_link" />
@@ -277,6 +279,7 @@
             <origin xyz="0.00563134 0.0 0.04718515" rpy="0 0 0" />
             <mimic joint="${prefix}robotiq_85_left_knuckle_joint" multiplier="-1" />
-        </joint>
-        <joint name="${prefix}robotiq_85_right_finger_tip_joint" type="continuous">
+            <limit lower="-0.8" upper="0.0" velocity="0.5" effort="50" />
+        </joint>
+        <joint name="${prefix}robotiq_85_right_finger_tip_joint" type="revolute">
             <parent link="${prefix}robotiq_85_right_finger_link" />
             <child link="${prefix}robotiq_85_right_finger_tip_link" />
@@ -284,4 +287,5 @@
             <origin xyz="-0.00563134 0.0 0.04718515" rpy="0 0 0" />
             <mimic joint="${prefix}robotiq_85_left_knuckle_joint" />
+            <limit lower="0.0" upper="0.8" velocity="0.5" effort="50" />
         </joint>
     </xacro:macro>
